Commit message: Modify Hardware INterface

File: src/uds_description/urdf/body/uds_base.urdf.xacro (robot description, xacro)
@@ -13,5 +13,5 @@
         <visual>
             <geometry>
-                <mesh filename="file://$(find uds_description)/meshes/assembled.stl" scale="0.001 0.001 0.001"/>
+                <mesh filename="package://uds_description/meshes/assembled.stl" scale="0.001 0.001 0.001"/>
             </geometry>
             <origin xyz="0 0 0" rpy="0 0 ${pi/2}"/>

File: src/uds_description/urdf/body/uds_robot.urdf.xacro (robot description, xacro)
@@ -9,7 +9,7 @@
     <xacro:include filename="$(find uds_description)/urdf/body/uds_wheel.urdf.xacro"/>
     <xacro:include filename="$(find uds_description)/urdf/body/uds_castor.urdf.xacro"/>
-    <xacro:include filename="$(find uds_description)/urdf/gazebo/gazebo_control.xacro"/>
+    <!-- <xacro:include filename="$(find uds_description)/urdf/gazebo/gazebo_control.xacro"/>  -->
     <!-- <xacro:include filename="$(find uds_description)/urdf/gazebo/uds.gazebo.xacro"/> -->
-    <!-- <xacro:include filename="$(find uds_description)/urdf/ros2_control/uds_ros2_control.xacro"/> -->
+    <xacro:include filename="$(find uds_description)/urdf/ros2_control/uds_ros2_control.xacro"/>
     <!-- <xacro:include filename="$(find uds_description)/urdf/sensors/rgbd_camera.urdf.xacro"/>
     <xacro:include filename="$(find uds_description)/urdf/sensors/imu.urdf.xacro"/> -->

File: src/uds_description/urdf/ros2_control/uds_ros2_control.xacro (robot description, xacro)
@@ -5,5 +5,5 @@
       <ros2_control name="RealRobot" type="system">
           <hardware>
-              <plugin>uds_hardware/UdsHardware</plugin>
+              <plugin>uds_hardware/DiffDriveUdsHardware</plugin>
               <param name="left_wheel_name">left_wheel_joint</param>
               <param name="right_wheel_name">right_wheel_joint</param>
@@ -11,6 +11,6 @@
               <param name="device">/dev/ttyUSB0</param>
               <param name="baud_rate">57600</param>
-              <param name="timeout">1000</param>
-              <param name="enc_counts_per_rev">3436</param>
+              <param name="timeout_ms">1000</param>
+              <param name="enc_counts_per_rev">1040</param>
           </hardware>
           <joint name="left_wheel_joint">
@@ -19,6 +19,6 @@
                   <param name="max">10</param>
               </command_interface>
+              <state_interface name="position"/>
               <state_interface name="velocity"/>
-              <state_interface name="position"/>
           </joint>
           <joint name="right_wheel_joint">
@@ -27,6 +27,6 @@
                   <param name="max">10</param>
               </command_interface>
+              <state_interface name="position"/>
               <state_interface name="velocity"/>
-              <state_interface name="position"/>
           </joint>
       </ros2_control>
